File: CC2652_OnBoard.kicad_pcb (KiCad board)
At the start: 2 copper layers, 66 parts, among them IC1 CC2652R1FRGZR, IC2 TLE493DW2B6A2HTSA1

Commit message: Update+UL PCB
Parts:
- removed FLASH_MEM1: W25Q32JVZP, Package_SON:WSON-8-1EP_6x5mm_P1.27mm_EP3.4x4.3mm
- removed Giroscope1: MPU-6050(I2C), Sensor_Motion:InvenSense_QFN-24_4x4mm_P0.5mm
- added EMI_VDDS_FILTER_USB1: BLM18HE152SN1D, Inductor_SMD:L_0603_1608Metric, F.Cu at (155.9, 85.5)
- added FLASH 64MB: W25Q64JWZPIM, Package_SON:WSON-8-1EP_6x5mm_P1.27mm_EP3.4x4.3mm, F.Cu at (102.5, 96.6)
- added MPU6050: MPU-6050(I2C), Sensor_Motion:InvenSense_QFN-24_4x4mm_P0.5mm, F.Cu at (121.4, 65.2)
- added REF**: MountingHole_3mm, MountingHole:MountingHole_3mm, F.Cu at (157.8, 50.0)
- added REF**: MountingHole_3mm, MountingHole:MountingHole_3mm, F.Cu at (157.8, 114.8)
- added REF**: MountingHole_3mm, MountingHole:MountingHole_3mm, F.Cu at (75.2, 114.8)
- added REF**: MountingHole_3mm, MountingHole:MountingHole_3mm, F.Cu at (75.2, 50.0)
- added REF**: Texas_SWRA117D_2.4GHz_Left, RF_Antenna:Texas_SWRA117D_2.4GHz_Left, F.Cu at (80.2, 80.5)
- Hall 3D: renamed from IC2
- JTAG XDS110: renamed from JTAG_DEBUG_HEADER1
- LED 1: renamed from LED_ROJO1
- LED 2: renamed from LED_VERDE1
- moved BTN2 160.8 mm to (146.3, 113.9)
- moved PINS_DER1 155.1 mm to (119.5, 113.5), turned to 270 degrees
- moved JTAG XDS110 148.6 mm to (149.4, 96.4), turned to 180 degrees
- moved BTN1 143.2 mm to (131.6, 114.0)
- moved BTN2_R1 142.4 mm to (148.1, 106.4), turned to 270 degrees
- moved BTN1_R1 130.8 mm to (132.0, 107.1), turned to 270 degrees
- moved RST 124.5 mm to (147.6, 50.7)
- moved PINS_PWR_DER1 118.5 mm to (89.6, 116.1), turned to 270 degrees
- moved R_RESET1 116.7 mm to (148.1, 57.0), turned to 90 degrees
- moved EMI_VDDS_FILTER1 112.3 mm to (149.3, 88.5)
- moved PINS_IZQ1 111.1 mm to (119.5, 49.2), turned to 270 degrees
- moved HALL_SCL_PUR1 108.4 mm to (132.4, 66.9)
- moved FLASH_nCS_PUR1 105.9 mm to (97.0, 94.9), turned to 270 degrees
- moved USB_UART1 104.7 mm to (146.8, 82.4), turned to 180 degrees
- moved HALL_SDA_PUR1 104.5 mm to (132.4, 64.2)
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- renumbered BTN_RST1 to RST, D_Rx1 to Rx, D_Tx1 to Tx
Connections:
- C110 pad 1: Net-(C110-Pad1) -> VDDS
- IC1 pad 15: FLASH_SDI -> FLASH_CLK
- IC1 pad 16: FLASH_CLK -> FLASH_SDI
- IC1 pad 28: GPIO18 -> CP2102_TX
- IC1 pad 29: GPIO19 -> CP2102_RX
- JTAG_ESD1 pad 1: RESET_N -> JTAG_TMSC
- JTAG_ESD1 pad 2: GPIO17-JTDI -> Net-(JTAG_ESD1-Pad2)
- JTAG_ESD1 pad 3: GPIO16-JTDO -> RESET_N
- JTAG_ESD1 pad 5: JTAG_TCKC -> GPIO17-JTDI
- JTAG_ESD1 pad 6: JTAG_TMSC -> GPIO16-JTDO
- JTAG_ESD1 pad 7: Net-(JTAG_ESD1-Pad7) -> JTAG_TCKC
- PINS_DER1 pad 12: FLASH_SDI -> Net-(PINS_DER1-Pad12)
- PINS_DER1 pad 14: FLASH_SDO -> Net-(PINS_DER1-Pad14)
- PINS_DER1 pad 5: FLASH_nCS -> Net-(PINS_DER1-Pad5)
- PINS_DER1 pad 7: GPIO19 -> Net-(PINS_DER1-Pad7)
- PINS_DER1 pad 9: GPIO18 -> Net-(PINS_DER1-Pad9)
- PINS_IZQ1 pad 13: FLASH_CLK -> Net-(PINS_IZQ1-Pad13)
- RST pad 1: Net-(BTN_RST1-Pad1) -> GND
- RST pad 2: GND -> Net-(BTN_RST1-Pad2)
- R_RESET1 pad 2: Net-(BTN_RST1-Pad1) -> Net-(BTN_RST1-Pad2)
- USB_CONNECTOR_A1 pad 1: USB_VBUS -> Net-(EMI_VDDS_FILTER_USB1-Pad2)
- USB_ESD1 pad 1: Net-(USB_ESD1-Pad1) -> USB_D-
- USB_ESD1 pad 3: Net-(USB_ESD1-Pad3) -> USB_D+
- USB_ESD1 pad 5: USB_D- -> Net-(USB_ESD1-Pad5)
- USB_ESD1 pad 6: USB_D+ -> Net-(USB_ESD1-Pad6)
Routing:
- net RESET_N: track 0.00 -> 148.5 mm, vias 0 -> 4
- net USB_VBUS: track 0.00 -> 105.4 mm, vias 0 -> 2
- net GPIO17-JTDI: track 0.00 -> 97.7 mm, vias 0 -> 3
- net GPIO16-JTDO: track 0.00 -> 97.2 mm, vias 0 -> 3
- net GPIO21: track 0.00 -> 95.4 mm
- net JTAG_TCKC: track 0.00 -> 93.9 mm, vias 0 -> 3
- net JTAG_TMSC: track 0.00 -> 92.4 mm, vias 0 -> 3
- net GPIO2: track 0.00 -> 89.3 mm, vias 0 -> 1
- net GPIO22: track 0.00 -> 85.0 mm
- net GPIO3: track 0.00 -> 84.5 mm, vias 0 -> 1
- net GPIO14: track 0.00 -> 79.8 mm
- net GPIO0: track 0.00 -> 74.7 mm, vias 0 -> 1
- net GPIO7: track 0.00 -> 73.2 mm
- net GPIO25: track 0.00 -> 72.9 mm, vias 0 -> 2
- net GPIO6: track 0.00 -> 71.7 mm, vias 0 -> 2
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- added copper zone on B.Cu, net GND
- added copper zone on F.Cu, net GND
- added copper zone on In1.Cu, net GND
- added copper zone on In2.Cu, net VDDS
Other:
- board outline added: 93.2 x 75.2 mm
- copper layers 2 -> 4
- net class Default: clearance 0.2 -> 0.127; trace_width 0.25 -> 0.127; via_dia 0.8 -> 0.4; via_drill 0.4 -> 0.2
- rule trace_clearance: 0.2 -> 0.127
- rule trace_min: 0.2 -> 0.127
- rule via_min_drill: 0.3 -> 0.2
- board text added: "GPIO13"
- board text added: "GPIO14"
- board text added: "GPIO6"
- board text added: "GPIO7"

Commit message: V2 PIN Route
Parts:
- D Rx: renamed from Rx
- D Tx: renamed from Tx
- FLASH_MEM: renamed from FLASH 64MB
- Hall: renamed from Hall 3D
- JTAG_DEBUG_HEADER1: renamed from JTAG XDS110
- LED_ROJO: renamed from LED 1
- LED_VERDE: renamed from LED 2
- moved EMI_VDDS_FILTER1 14.0 mm to (137.7, 80.8)
- moved R_LED_VERDE1 9.45 mm to (93.2, 102.8), turned to 270 degrees
- moved R_LED_ROJO1 8.39 mm to (90.8, 102.8), turned to 270 degrees
- moved LED_VERDE 5.95 mm to (93.2, 98.8), turned to 90 degrees
- moved LED_ROJO 3.03 mm to (90.8, 98.8), turned to 90 degrees
- moved 32KHz_Crystl1 2.28 mm to (95.1, 84.0)
- moved C1 2.28 mm to (92.3, 82.8)
- moved C2 2.28 mm to (92.3, 85.2)
- moved C111 1.30 mm to (136.8, 61.1)
- renumbered RST to BTN_RST1, MPU6050 to Giroscope
Connections:
- PINS_DER1 pad 1: GPIO7 -> GPIO16-JTDO
- PINS_DER1 pad 10: RESET_N -> GPIO11
- PINS_DER1 pad 11: Net-(PINS_DER1-Pad11) -> GPIO7
- PINS_DER1 pad 12: Net-(PINS_DER1-Pad12) -> GPIO6
- PINS_DER1 pad 13: JTAG_TMSC -> GND
- PINS_DER1 pad 14: Net-(PINS_DER1-Pad14) -> GND
- PINS_DER1 pad 15: JTAG_TCKC -> GPIO5
- PINS_DER1 pad 16: GPIO13 -> GPIO4
- PINS_DER1 pad 17: GPIO16-JTDO -> GPIO3
- PINS_DER1 pad 18: GPIO14 -> GPIO2
- PINS_DER1 pad 19: GPIO17-JTDI -> GPIO1
- PINS_DER1 pad 2: GND -> GPIO17-JTDI
- PINS_DER1 pad 20: GPIO15 -> GPIO0
- PINS_DER1 pad 3: GPIO6 -> JTAG_TMSC
- PINS_DER1 pad 4: GPIO12 -> JTAG_TCKC
- PINS_DER1 pad 5: Net-(PINS_DER1-Pad5) -> GPIO15
- PINS_DER1 pad 6: GPIO11 -> GPIO14
- PINS_DER1 pad 7: Net-(PINS_DER1-Pad7) -> GND
- PINS_DER1 pad 8: Net-(PINS_DER1-Pad8) -> GPIO13
- PINS_DER1 pad 9: Net-(PINS_DER1-Pad9) -> GPIO12
- PINS_IZQ1 pad 1: VDDS -> USB_VBUS
- PINS_IZQ1 pad 10: GPIO27 -> GPIO23
- PINS_IZQ1 pad 11: GPIO24 -> GND
- PINS_IZQ1 pad 12: GPIO28 -> GPIO26
- PINS_IZQ1 pad 13: Net-(PINS_IZQ1-Pad13) -> GND
- PINS_IZQ1 pad 14: GPIO29 -> GPIO27
- PINS_IZQ1 pad 15: GPIO21 -> GND
- PINS_IZQ1 pad 16: GPIO30 -> GPIO28
- PINS_IZQ1 pad 17: GPIO4 -> GND
- PINS_IZQ1 pad 18: GPIO0 -> GPIO29
- PINS_IZQ1 pad 19: GPIO5 -> GND
- PINS_IZQ1 pad 2: USB_VBUS -> GPIO24
- PINS_IZQ1 pad 20: GPIO1 -> GPIO30
- PINS_IZQ1 pad 3: GPIO23 -> GND
- PINS_IZQ1 pad 4: GND -> GPIO25
- PINS_IZQ1 pad 5: GPIO2 -> GND
- PINS_IZQ1 pad 6: GPIO25 -> GPIO21
- PINS_IZQ1 pad 7: GPIO3 -> GND
- PINS_IZQ1 pad 8: GPIO26 -> GPIO22
- PINS_IZQ1 pad 9: GPIO22 -> GND
Routing:
- net RESET_N: track 148.5 -> 91.0 mm, vias 4 -> 2
- net GPIO21: track 95.4 -> 53.3 mm, vias 0 -> 1
- net GPIO2: track 89.3 -> 51.4 mm, vias 1 -> 0
- net GPIO3: track 84.5 -> 49.1 mm, vias 1 -> 0
- net GPIO22: track 85.0 -> 50.5 mm, vias 0 -> 1
- net GPIO7: track 73.2 -> 40.3 mm
- net FLASH_nCS: track 25.3 -> 49.6 mm
- net GPIO0: track 74.7 -> 50.5 mm, vias 1 -> 0
- net GPIO1: track 70.5 -> 47.8 mm, vias 1 -> 0
- net GPIO6: track 71.7 -> 49.4 mm, vias 2 -> 0
- net Vin_CC2652: track 45.6 -> 66.4 mm, vias 5 -> 3
- net GPIO4: track 69.4 -> 52.0 mm, vias 1 -> 0
- net GPIO17-JTDI: track 97.7 -> 81.1 mm, vias 3 -> 1
- net GPIO16-JTDO: track 97.2 -> 80.5 mm, vias 3 -> 1
- net GPIO24: track 70.6 -> 55.6 mm
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Other:
- net class Default: via_dia 0.4 -> 0.45
- rule via_min_size: 0.4 -> 0.45
- board text added: "---------T---------"
- board text added: "0"
- board text added: "1"
- board text added: "11"
- board text added: "12"
- board text added: "13"
- board text added: "14"
- board text added: "15"
- board text added: "2"
- board text added: "21"
- board text added: "22"
- board text added: "23"
- board text added: "24"
- board text added: "25"
- board text added: "26"
- board text added: "27"
- board text added: "28"
- board text added: "29"
- board text added: "3"
- board text added: "3.3V"
- board text added: "30"
- board text added: "4"
- board text added: "5"
- board text added: "5V"
- board text added: "6"
- board text added: "7"
- board text added: "JTDO"
- board text added: "T"
- board text added: "TCKC/JTDI"
- board text added: "TMSC"
